File: sensor_pcb/sensor_pcb.sch (KiCad schematic (older format))
At the start: 53 parts, among them J1 AVR-ISP-6, J2 SMA female, J3 Arc, J4 Arc, Q1 AO3401A, Q2 AO3401A, U1 MCP1700-3302E_SOT23, U2 HIH6131-021-001, U3 ATmega328P-AU, Y1 8 MHz

Commit message: Added sensor case
Parts:
- J2: footprint Connector_Coaxial:SMA_Samtec_SMA-J-P-X-ST-EM1_EdgeMount -> sensor_pcb:SMA_Samtec_SMA-J-P-X-ST-EM1_EdgeMount
Changed lines of the file:
@@
 F 0 "J2" H 10800 1975 50  0000 R CNN
 F 1 "SMA female" H 10800 1875 50  0000 R CNN
-F 2 "Connector_Coaxial:SMA_Samtec_SMA-J-P-X-ST-EM1_EdgeMount" H 10925 1950 60  0001 L CNN
+F 2 "sensor_pcb:SMA_Samtec_SMA-J-P-X-ST-EM1_EdgeMount" H 10925 1950 60  0001 L CNN
 F 3 "http://www.belfuse.com/resources/Johnson/drawings/dr-1420701801.pdf" H 10925 2050 60  0001 L CNN
 F 4 "J502-ND" H 10925 2150 60  0001 L CNN "Digi-Key_PN"
