File: scanner_circuit/scanner_circuit.sch (KiCad schematic (older format))
At the start: 39 parts, among them Q1 2N7000, Q2 IRF9540N, SW1 Red_Button, SW2 Blue_Button, SW3 Green_Button, U1 ATmega328P-PU, U2 LoRa Shield, U3 LD1117S33TR_SOT223, U4 LM317_TO220, Y1 Crystal

Commit message: Added footprints to TTN mapper
Parts:
- BT1: footprint (none) -> STRIP_100MIL2
- C1, C2, C4, C5, C6, C8: footprint (none) -> CAP_CERAMIC
- C3, C7, C9: footprint (none) -> CAP_ELECTRO_200
- Q1: footprint Package_TO_SOT_THT:TO-92_Inline -> TO92
- Q2, U4: footprint Package_TO_SOT_THT:TO-220-3_Vertical -> TO220
- R1, R10, R11, R12, R13, R14, R2, R3, R4, R5, R6, R7, R8, R9: footprint (none) -> RESISTOR
- RV1: footprint (none) -> TRIM_VERT
- U3: footprint Package_TO_SOT_SMD:SOT-223-3_TabPin2 -> TO220
- Y1: value Crystal -> 16 MHz
- Z1: footprint Diode_THT:D_DO-41_SOD81_P10.16mm_Horizontal -> DIODE
- gave numbers to parts that had none: 1
Changed lines of the file:
@@
 F 0 "C3" H 4538 1321 50  0000 L CNN
 F 1 "47uF" H 4538 1230 50  0000 L CNN
-F 2 "" H 4450 1275 50  0001 C CNN
+F 2 "CAP_ELECTRO_200" H 4450 1275 50  0001 C CNN
 F 3 "~" H 4450 1275 50  0001 C CNN
 	1    4450 1275
@@
 F 0 "C4" H 4117 1321 50  0000 L CNN
 F 1 "100nF" H 4117 1230 50  0000 L CNN
-F 2 "" H 4025 1275 50  0001 C CNN
+F 2 "CAP_CERAMIC" H 4025 1275 50  0001 C CNN
 F 3 "~" H 4025 1275 50  0001 C CNN
 	1    4025 1275
@@
 F 0 "C2" H 5717 2746 50  0000 L CNN
 F 1 "22pF" H 5717 2655 50  0000 L CNN
-F 2 "" H 5625 2700 50  0001 C CNN
+F 2 "CAP_CERAMIC" H 5625 2700 50  0001 C CNN
 F 3 "~" H 5625 2700 50  0001 C CNN
 	1    5625 2700
@@
 F 0 "Q1" V 6325 6050 50  0000 L CNN
 F 1 "2N7000" V 6425 6050 50  0000 L CNN
-F 2 "Package_TO_SOT_THT:TO-92_Inline" H 6325 6125 50  0001 L CIN
+F 2 "TO92" H 6325 6125 50  0001 L CIN
 F 3 "https://www.fairchildsemi.com/datasheets/2N/2N7000.pdf" H 6125 6200 50  0001 L CNN
 	1    6125 6200
@@
 F 0 "R1" H 5934 5971 50  0000 L CNN
 F 1 "10k" H 5934 5880 50  0000 L CNN
-F 2 "" H 5875 5925 50  0001 C CNN
+F 2 "RESISTOR" H 5875 5925 50  0001 C CNN
 F 3 "~" H 5875 5925 50  0001 C CNN
 	1    5875 5925
@@
 F 0 "R2" H 6434 5971 50  0000 L CNN
 F 1 "10k" H 6434 5880 50  0000 L CNN
-F 2 "" H 6375 5925 50  0001 C CNN
+F 2 "RESISTOR" H 6375 5925 50  0001 C CNN
 F 3 "~" H 6375 5925 50  0001 C CNN
 	1    6375 5925
@@
 F 0 "R12" V 1643 4075 50  0000 C CNN
 F 1 "620R" V 1734 4075 50  0000 C CNN
-F 2 "" V 1780 4075 50  0001 C CNN
+F 2 "RESISTOR" V 1780 4075 50  0001 C CNN
 F 3 "~" H 1850 4075 50  0001 C CNN
 	1    1850 4075
@@
 F 0 "R11" V 1643 3625 50  0000 C CNN
 F 1 "120R" V 1734 3625 50  0000 C CNN
-F 2 "" V 1780 3625 50  0001 C CNN
+F 2 "RESISTOR" V 1780 3625 50  0001 C CNN
 F 3 "~" H 1850 3625 50  0001 C CNN
 	1    1850 3625
@@
 F 0 "R10" V 1643 3275 50  0000 C CNN
 F 1 "120R" V 1734 3275 50  0000 C CNN
-F 2 "" V 1780 3275 50  0001 C CNN
+F 2 "RESISTOR" V 1780 3275 50  0001 C CNN
 F 3 "~" H 1850 3275 50  0001 C CNN
 	1    1850 3275
@@
 F 0 "R13" V 1643 4425 50  0000 C CNN
 F 1 "120R" V 1734 4425 50  0000 C CNN
-F 2 "" V 1780 4425 50  0001 C CNN
+F 2 "RESISTOR" V 1780 4425 50  0001 C CNN
 F 3 "~" H 1850 4425 50  0001 C CNN
 	1    1850 4425
@@
 F 0 "C9" V 2450 3250 50  0000 C CNN
 F 1 "10uF" V 2359 3250 50  0000 C CNN
-F 2 "" H 2225 3250 50  0001 C CNN
+F 2 "CAP_ELECTRO_200" H 2225 3250 50  0001 C CNN
 F 3 "~" H 2225 3250 50  0001 C CNN
 	1    2225 3250
@@
 F 0 "R8" V 9568 2650 50  0000 C CNN
 F 1 "20k" V 9659 2650 50  0000 C CNN
-F 2 "" V 9705 2650 50  0001 C CNN
+F 2 "RESISTOR" V 9705 2650 50  0001 C CNN
 F 3 "~" H 9775 2650 50  0001 C CNN
 	1    9775 2650
@@
 F 0 "R6" V 9568 3400 50  0000 C CNN
 F 1 "10k" V 9659 3400 50  0000 C CNN
-F 2 "" V 9705 3400 50  0001 C CNN
+F 2 "RESISTOR" V 9705 3400 50  0001 C CNN
 F 3 "~" H 9775 3400 50  0001 C CNN
 	1    9775 3400
@@
 F 0 "R9" V 9918 3400 50  0000 C CNN
 F 1 "20k" V 10009 3400 50  0000 C CNN
-F 2 "" V 10055 3400 50  0001 C CNN
+F 2 "RESISTOR" V 10055 3400 50  0001 C CNN
 F 3 "~" H 10125 3400 50  0001 C CNN
 	1    10125 3400
@@
 F 0 "C6" V 1475 5775 50  0000 L CNN
 F 1 "100nF" V 1375 5725 50  0000 L CNN
-F 2 "" H 1225 5825 50  0001 C CNN
+F 2 "CAP_CERAMIC" H 1225 5825 50  0001 C CNN
 F 3 "~" H 1225 5825 50  0001 C CNN
 	1    1225 5825
@@
 F 0 "C8" V 1225 3175 50  0000 L CNN
 F 1 "100nF" V 1125 3125 50  0000 L CNN
-F 2 "" H 975 3225 50  0001 C CNN
+F 2 "CAP_CERAMIC" H 975 3225 50  0001 C CNN
 F 3 "~" H 975 3225 50  0001 C CNN
 	1    975  3225
@@
 F 0 "U4" H 1400 2783 50  0001 C CNN
 F 1 "LM317_TO220" H 1400 2874 50  0000 C CNN
-F 2 "Package_TO_SOT_THT:TO-220-3_Vertical" H 1400 2825 50  0001 C CIN
+F 2 "TO220" H 1400 2825 50  0001 C CIN
 F 3 "http://www.ti.com/lit/ds/symlink/lm337-n.pdf" H 1400 3025 50  0001 C CNN
 	1    1400 3025
@@
 F 0 "R7" V 9518 1900 50  0000 C CNN
 F 1 "68k" V 9609 1900 50  0000 C CNN
-F 2 "" V 9655 1900 50  0001 C CNN
+F 2 "RESISTOR" V 9655 1900 50  0001 C CNN
 F 3 "~" H 9725 1900 50  0001 C CNN
 	1    9725 1900
@@
 F 0 "R5" V 9518 1325 50  0000 C CNN
 F 1 "100k" V 9609 1325 50  0000 C CNN
-F 2 "" V 9655 1325 50  0001 C CNN
+F 2 "RESISTOR" V 9655 1325 50  0001 C CNN
 F 3 "~" H 9725 1325 50  0001 C CNN
 	1    9725 1325
@@
 F 0 "U3" H 1650 5792 50  0001 C CNN
 F 1 "LD1117S33TR_SOT223" H 1650 5701 50  0000 C CNN
-F 2 "Package_TO_SOT_SMD:SOT-223-3_TabPin2" H 1650 5750 50  0001 C CNN
+F 2 "TO220" H 1650 5750 50  0001 C CNN
 F 3 "http://www.st.com/st-web-ui/static/active/en/resource/technical/document/datasheet/CD00000544.pdf" H 1750 5300 50  0001 C CNN
 	1    1650 5550
@@
 F 0 "C7" H 2138 5871 50  0000 L CNN
 F 1 "10uF" H 2138 5780 50  0000 L CNN
-F 2 "" H 2050 5825 50  0001 C CNN
+F 2 "CAP_ELECTRO_200" H 2050 5825 50  0001 C CNN
 F 3 "~" H 2050 5825 50  0001 C CNN
 	1    2050 5825
@@
 F 0 "R3" V 4975 3050 50  0000 L CNN
 F 1 "10k" V 4775 3050 50  0000 L CNN
-F 2 "" H 4875 3100 50  0001 C CNN
+F 2 "RESISTOR" H 4875 3100 50  0001 C CNN
 F 3 "~" H 4875 3100 50  0001 C CNN
 	1    4875 3100
@@
 P 5225 2350
 F 0 "Y1" V 5179 2481 50  0000 L CNN
-F 1 "Crystal" V 5270 2481 50  0000 L CNN
+F 1 "16 MHz" V 5270 2481 50  0000 L CNN
 F 2 "" H 5225 2350 50  0001 C CNN
 F 3 "~" H 5225 2350 50  0001 C CNN
@@
 F 0 "C1" H 5317 2746 50  0000 L CNN
 F 1 "22pF" H 5317 2655 50  0000 L CNN
-F 2 "" H 5225 2700 50  0001 C CNN
+F 2 "CAP_CERAMIC" H 5225 2700 50  0001 C CNN
 F 3 "~" H 5225 2700 50  0001 C CNN
 	1    5225 2700
@@
 F 0 "Q2" V 1992 1250 50  0000 C CNN
 F 1 "IRF9540N" V 1901 1250 50  0000 C CNN
-F 2 "Package_TO_SOT_THT:TO-220-3_Vertical" H 1850 1175 50  0001 L CIN
+F 2 "TO220" H 1850 1175 50  0001 L CIN
 F 3 "http://www.irf.com/product-info/datasheets/data/irf9540n.pdf" H 1650 1250 50  0001 L CNN
 	1    1650 1250
@@
 F 0 "RV1" H 8505 1479 50  0000 R CNN
 F 1 "10k" H 8505 1570 50  0000 R CNN
-F 2 "" H 8575 1525 50  0001 C CNN
+F 2 "TRIM_VERT" H 8575 1525 50  0001 C CNN
 F 3 "~" H 8575 1525 50  0001 C CNN
 	1    8575 1525
@@
 F 0 "R14" V 1443 1800 50  0000 C CNN
 F 1 "100k" V 1534 1800 50  0000 C CNN
-F 2 "" V 1580 1800 50  0001 C CNN
+F 2 "RESISTOR" V 1580 1800 50  0001 C CNN
 F 3 "~" H 1650 1800 50  0001 C CNN
 	1    1650 1800
@@
 F 0 "Z1" H 2050 1616 50  0000 C CNN
 F 1 "10V" H 2050 1525 50  0000 C CNN
-F 2 "Diode_THT:D_DO-41_SOD81_P10.16mm_Horizontal" H 2050 1225 50  0001 C CNN
+F 2 "DIODE" H 2050 1225 50  0001 C CNN
 F 3 "http://www.vishay.com/docs/85790/zpy3v9.pdf" H 2050 1400 50  0001 C CNN
 	1    2050 1400
@@
 F 0 "BT1" H 825 1775 50  0000 L CNN
 F 1 "5x AA" H 750 1675 50  0000 L CNN
-F 2 "" V 1100 1735 50  0001 C CNN
+F 2 "STRIP_100MIL2" V 1100 1735 50  0001 C CNN
 F 3 "~" V 1100 1735 50  0001 C CNN
 	1    1100 1675
@@
 F 0 "C5" H 2967 2046 50  0000 L CNN
 F 1 "100nF" H 2967 1955 50  0000 L CNN
-F 2 "" H 2875 2000 50  0001 C CNN
+F 2 "CAP_CERAMIC" H 2875 2000 50  0001 C CNN
 F 3 "~" H 2875 2000 50  0001 C CNN
 	1    2875 2000
@@
 F 0 "R4" V 8075 1775 50  0000 L CNN
 F 1 "220R" V 7875 1675 50  0000 L CNN
-F 2 "" H 7975 1825 50  0001 C CNN
+F 2 "RESISTOR" H 7975 1825 50  0001 C CNN
 F 3 "~" H 7975 1825 50  0001 C CNN
 	1    7975 1825
@@
 $EndComp
 $Comp
-L Connector:AVR-ISP-6 J?
+L Connector:AVR-ISP-6 J1
 U 1 1 5DF97998
 P 10200 5725
-F 0 "J?" H 9871 5821 50  0000 R CNN
+F 0 "J1" H 9871 5821 50  0000 R CNN
 F 1 "AVR-ISP-6" H 9871 5730 50  0000 R CNN
 F 2 "" V 9950 5775 50  0001 C CNN
@@
 $EndComp
 $Comp
-L power:+5V #PWR?
+L power:+5V #PWR0119
 U 1 1 5DFA67B5
 P 10100 5175
-F 0 "#PWR?" H 10100 5025 50  0001 C CNN
+F 0 "#PWR0119" H 10100 5025 50  0001 C CNN
 F 1 "+5V" H 10115 5348 50  0000 C CNN
 F 2 "" H 10100 5175 50  0001 C CNN
@@
 $EndComp
 $Comp
-L power:GND #PWR?
+L power:GND #PWR0120
 U 1 1 5DFA6B8E
 P 10100 6175
-F 0 "#PWR?" H 10100 5925 50  0001 C CNN
+F 0 "#PWR0120" H 10100 5925 50  0001 C CNN
 F 1 "GND" H 10105 6002 50  0000 C CNN
 F 2 "" H 10100 6175 50  0001 C CNN

Commit message: Added perf board netlist
Parts:
- DS1: footprint Display:WC1602A -> STRIP_100MIL16
- ISP1: renamed from J1; footprint (none) -> ISP_CONNECTOR
- MOD1: footprint (none) -> STRIP_100MIL9
- MOD2: renamed from U2; footprint (none) -> LORA_SHIELD
- SW1, SW2, SW3: footprint (none) -> PUSH_BUTTON
- U1: footprint Package_DIP:DIP-28_W7.62mm -> DIP28
- Y1: footprint (none) -> XTAL_HC-49
Changed lines of the file:
@@
 F 0 "DS1" H 7825 825 50  0001 C CNN
 F 1 "LCD Screen" V 7225 1975 62  0000 C CNB
-F 2 "Display:WC1602A" H 7225 1225 50  0001 C CIN
+F 2 "STRIP_100MIL16" H 7225 1225 50  0001 C CIN
 F 3 "http://www.wincomlcd.com/pdf/WC1602A-SFYLYHTC06.pdf" H 7925 2125 50  0001 C CNN
 	1    7225 2125
@@
 F 0 "SW3" V 10475 3950 50  0001 R CNN
 F 1 "Green_Button" V 10375 4250 50  0000 R CNN
-F 2 "" H 10375 3800 50  0001 C CNN
+F 2 "PUSH_BUTTON" H 10375 3800 50  0001 C CNN
 F 3 "~" H 10375 3800 50  0001 C CNN
 	1    10375 3600
@@
 F 0 "SW2" V 10475 3200 50  0001 R CNN
 F 1 "Blue_Button" V 10375 3450 50  0000 R CNN
-F 2 "" H 10375 3050 50  0001 C CNN
+F 2 "PUSH_BUTTON" H 10375 3050 50  0001 C CNN
 F 3 "~" H 10375 3050 50  0001 C CNN
 	1    10375 2850
@@
 F 0 "SW1" V 10475 2450 50  0001 R CNN
 F 1 "Red_Button" V 10375 2650 50  0000 R CNN
-F 2 "" H 10375 2300 50  0001 C CNN
+F 2 "PUSH_BUTTON" H 10375 2300 50  0001 C CNN
 F 3 "~" H 10375 2300 50  0001 C CNN
 	1    10375 2100
@@
 F 0 "MOD1" H 9650 5325 50  0001 L CNN
 F 1 "GPS MODULE" V 8650 5425 71  0000 L CNB
-F 2 "" H 8750 5875 50  0001 C CNN
+F 2 "STRIP_100MIL9" H 8750 5875 50  0001 C CNN
 F 3 "" H 8750 5875 50  0001 C CNN
 	1    8750 5775
@@
 F 0 "U1" H 3081 3046 50  0001 R CNN
 F 1 "ATmega328P-PU" V 3525 3600 118 0000 R CNB
-F 2 "Package_DIP:DIP-28_W7.62mm" H 3725 3000 50  0001 C CIN
+F 2 "DIP28" H 3725 3000 50  0001 C CIN
 F 3 "http://ww1.microchip.com/downloads/en/DeviceDoc/ATmega328_P%20AVR%20MCU%20with%20picoPower%20Technology%20Data%20Sheet%2040001984A.pdf" H 3725 3000 50  0001 C CNN
 	1    3725 3000
@@
 F 0 "Y1" V 5179 2481 50  0000 L CNN
 F 1 "16 MHz" V 5270 2481 50  0000 L CNN
-F 2 "" H 5225 2350 50  0001 C CNN
+F 2 "XTAL_HC-49" H 5225 2350 50  0001 C CNN
 F 3 "~" H 5225 2350 50  0001 C CNN
 	1    5225 2350
@@
 D10
 $Comp
-L scanner_components:dragino_lora_shield U2
+L scanner_components:dragino_lora_shield MOD2
 U 1 1 5DEF3113
 P 3400 5500
-F 0 "U2" H 3450 5500 50  0001 L CNN
+F 0 "MOD2" H 3450 5500 50  0001 L CNN
 F 1 "LoRa Shield" H 3850 6150 58  0000 L CNB
-F 2 "" H 3400 6250 50  0001 C CNN
+F 2 "LORA_SHIELD" H 3400 6250 50  0001 C CNN
 F 3 "" H 3400 6250 50  0001 C CNN
 	1    3400 5500
@@
 $EndComp
 $Comp
-L Connector:AVR-ISP-6 J1
+L Connector:AVR-ISP-6 ISP1
 U 1 1 5DF97998
 P 10200 5725
-F 0 "J1" H 9871 5821 50  0000 R CNN
+F 0 "ISP1" H 9871 5821 50  0000 R CNN
 F 1 "AVR-ISP-6" H 9871 5730 50  0000 R CNN
-F 2 "" V 9950 5775 50  0001 C CNN
+F 2 "ISP_CONNECTOR" V 9950 5775 50  0001 C CNN
 F 3 " ~" H 8925 5175 50  0001 C CNN
 	1    10200 5725

Commit message: Changed resistor values in scanner circuit
Parts:
- R12: value 620R -> 470R
- R13: value 120R -> 270R
Changed lines of the file:
@@
 P 1850 4075
 F 0 "R12" V 1643 4075 50  0000 C CNN
-F 1 "620R" V 1734 4075 50  0000 C CNN
+F 1 "470R" V 1734 4075 50  0000 C CNN
 F 2 "RESISTOR" V 1780 4075 50  0001 C CNN
 F 3 "~" H 1850 4075 50  0001 C CNN
@@
 P 1850 4425
 F 0 "R13" V 1643 4425 50  0000 C CNN
-F 1 "120R" V 1734 4425 50  0000 C CNN
+F 1 "270R" V 1734 4425 50  0000 C CNN
 F 2 "RESISTOR" V 1780 4425 50  0001 C CNN
 F 3 "~" H 1850 4425 50  0001 C CNN
